Commit message: added new rtab node and launch file, and updated to urdf modulet to contain neccessary sensor to perform SLAM w/ RTAB

File: my_robot/urdf/my_robot.xacro (robot description, xacro)
@@ -28,4 +28,11 @@
     <axis xyz="0 1 0" rpy="0 0 0"/>
   </joint>
+  <!-- Additional Camera for Rtab-SLAM -->
+  <!-- this is a child of the original camera link -->
+  <joint name="camera_optical_joint" type="fixed">
+    <origin xyz="0 0 0" rpy="-1.5707 0 -1.5707"/>
+    <parent link="camera"/>
+    <child link="camera_link_optical"/>
+  </joint>
   <link name='camera'>
     <pose>0 0 0 0 0 0</pose>
@@ -56,4 +63,6 @@
     </visual>
   </link>
+  <link name="camera_link_optical">
+  </link>
   <link name='hokuyo'>
     <pose>0 0 0 0 0 0</pose>
